Commit message: Change int to float in velocity

File: urdf/dbot.urdf.xacro (robot description, xacro)
@@ -99,5 +99,5 @@
         <child link="j0_link"/>
         <axis xyz="0 0 1"/>
-        <limit lower="${-pi}" upper="${pi}" velocity="100" effort="100"/>
+        <limit lower="${-pi}" upper="${pi}" velocity="100.0" effort="100.0"/>
     </joint>
     <!-- The j0 link of the robot -->
@@ -123,5 +123,5 @@
         <child link="j1_link"/>
         <axis xyz="0 0 1"/>
-        <limit lower="${-pi}" upper="${pi}" velocity="100" effort="100"/>
+        <limit lower="${-pi}" upper="${pi}" velocity="100.0" effort="100.0"/>
     </joint>
     <!-- The j1 link of the robot -->
@@ -160,5 +160,5 @@
         <child link="j2_link"/>
         <axis xyz="0 0 1"/>
-        <limit lower="${-pi}" upper="${pi}" velocity="100" effort="100"/>
+        <limit lower="${-pi}" upper="${pi}" velocity="100.0" effort="100.0"/>
     </joint>
     <!-- The j2 link of the robot -->
@@ -197,5 +197,5 @@
         <child link="j3_link"/>
         <axis xyz="0 0 1"/>
-        <limit lower="${-pi}" upper="${pi}" velocity="100" effort="100"/>
+        <limit lower="${-pi}" upper="${pi}" velocity="100.0" effort="100.0"/>
     </joint>
     <!-- The j3 link of the robot -->
@@ -221,5 +221,5 @@
         <child link="j4_link"/>
         <axis xyz="0 0 1"/>
-        <limit lower="${-pi}" upper="${pi}" velocity="100" effort="100"/>
+        <limit lower="${-pi}" upper="${pi}" velocity="100.0" effort="100.0"/>
     </joint>
     <!-- The j4 link of the robot -->
@@ -245,5 +245,5 @@
         <child link="j5_link"/>
         <axis xyz="0 0 1"/>
-        <limit lower="${-2*pi}" upper="${2*pi}" velocity="100" effort="100"/>
+        <limit lower="${-2*pi}" upper="${2*pi}" velocity="100.0" effort="100.0"/>
     </joint>
     <!-- The j5 link of the robot -->

Commit message: Add dynamics tag

File: urdf/dbot.urdf.xacro (robot description, xacro)
@@ -76,4 +76,6 @@
     <xacro:property name="flange_xyz" value="0.0 0.0 ${-flange_l/2}" />
     <xacro:property name="flange_rpy" value="0.0 0.0 0.0" />
+    <xacro:property name="damping" value="10.0" />
+    <xacro:property name="friction" value="10.0" />
     <!-- The first link of the robot -->
     <!-- Fixed base-->
@@ -92,4 +94,7 @@
             </geometry>
         </collision>
+        <xacro:inertial_cylinder mass="1.0" length="${base_l}" radius="${base_r}">
+            <origin xyz="${base_xyz}" rpy="${base_rpy}"/>
+        </xacro:inertial_cylinder>
     </link>
     <!-- Base to j0 -->
@@ -99,5 +104,6 @@
         <child link="j0_link"/>
         <axis xyz="0 0 1"/>
-        <limit lower="${-pi}" upper="${pi}" velocity="100.0" effort="100.0"/>
+        <limit lower="${-pi}" upper="${pi}" velocity="100" effort="100"/>
+        <dynamics damping="${damping}" friction="${friction}" />
     </joint>
     <!-- The j0 link of the robot -->
@@ -116,4 +122,7 @@
             </geometry>
         </collision>
+        <xacro:inertial_cylinder mass="1.0" length="${j0_l}" radius="${j0_r}">
+            <origin xyz="${j0_xyz}" rpy="${j0_rpy}"/>
+        </xacro:inertial_cylinder>
     </link>
     <!-- j0 to j1 Joint -->
@@ -123,5 +132,6 @@
         <child link="j1_link"/>
         <axis xyz="0 0 1"/>
-        <limit lower="${-pi}" upper="${pi}" velocity="100.0" effort="100.0"/>
+        <limit lower="${-pi}" upper="${pi}" velocity="100" effort="100"/>
+        <dynamics damping="${damping}" friction="${friction}" />
     </joint>
     <!-- The j1 link of the robot -->
@@ -140,4 +150,7 @@
             </geometry>
         </collision>
+        <xacro:inertial_cylinder mass="1.0" length="${j1_l}" radius="${j1_r}">
+            <origin xyz="${j1_xyz}" rpy="${j1_rpy}"/>
+        </xacro:inertial_cylinder>
         <visual>
             <origin xyz="${j1_link_xyz}" rpy="${j1_link_rpy}"/>
@@ -153,4 +166,7 @@
             </geometry>
         </collision>
+        <xacro:inertial_cylinder mass="1.0" length="${j1_link_l}" radius="${j1_link_r}">
+            <origin xyz="${j1_link_xyz}" rpy="${j1_link_rpy}"/>
+        </xacro:inertial_cylinder>
     </link>
     <!-- j1 to j2 Joint -->
@@ -160,5 +176,6 @@
         <child link="j2_link"/>
         <axis xyz="0 0 1"/>
-        <limit lower="${-pi}" upper="${pi}" velocity="100.0" effort="100.0"/>
+        <limit lower="${-pi}" upper="${pi}" velocity="100" effort="100"/>
+        <dynamics damping="${damping}" friction="${friction}" />
     </joint>
     <!-- The j2 link of the robot -->
@@ -177,4 +194,7 @@
             </geometry>
         </collision>
+        <xacro:inertial_cylinder mass="1.0" length="${j2_l}" radius="${j2_r}">
+            <origin xyz="${j2_xyz}" rpy="${j2_rpy}"/>
+        </xacro:inertial_cylinder>
         <visual>
             <origin xyz="${j2_link_xyz}" rpy="${j2_link_rpy}"/>
@@ -190,4 +210,7 @@
             </geometry>
         </collision>
+        <xacro:inertial_cylinder mass="1.0" length="${j2_link_l}" radius="${j2_link_r}">
+            <origin xyz="${j2_link_xyz}" rpy="${j2_link_rpy}"/>
+        </xacro:inertial_cylinder>
     </link>
     <!-- j2 to j3 Joint -->
@@ -197,5 +220,6 @@
         <child link="j3_link"/>
         <axis xyz="0 0 1"/>
-        <limit lower="${-pi}" upper="${pi}" velocity="100.0" effort="100.0"/>
+        <limit lower="${-pi}" upper="${pi}" velocity="100" effort="100"/>
+        <dynamics damping="${damping}" friction="${friction}" />
     </joint>
     <!-- The j3 link of the robot -->
@@ -214,4 +238,7 @@
             </geometry>
         </collision>
+        <xacro:inertial_cylinder mass="1.0" length="${j3_l}" radius="${j3_r}">
+            <origin xyz="${j3_xyz}" rpy="${j3_rpy}"/>
+        </xacro:inertial_cylinder>
     </link>
     <!-- j3 to j4 Joint -->
@@ -221,5 +248,6 @@
         <child link="j4_link"/>
         <axis xyz="0 0 1"/>
-        <limit lower="${-pi}" upper="${pi}" velocity="100.0" effort="100.0"/>
+        <limit lower="${-pi}" upper="${pi}" velocity="100" effort="100"/>
+        <dynamics damping="${damping}" friction="${friction}" />
     </joint>
     <!-- The j4 link of the robot -->
@@ -238,4 +266,7 @@
             </geometry>
         </collision>
+        <xacro:inertial_cylinder mass="1.0" length="${j4_l}" radius="${j4_r}">
+            <origin xyz="${j4_xyz}" rpy="${j4_rpy}"/>
+        </xacro:inertial_cylinder>
     </link>
     <!-- j4 to j5 Joint -->
@@ -245,5 +276,6 @@
         <child link="j5_link"/>
         <axis xyz="0 0 1"/>
-        <limit lower="${-2*pi}" upper="${2*pi}" velocity="100.0" effort="100.0"/>
+        <limit lower="${-2*pi}" upper="${2*pi}" velocity="100" effort="100"/>
+        <dynamics damping="${damping}" friction="${friction}" />
     </joint>
     <!-- The j5 link of the robot -->
@@ -262,4 +294,7 @@
             </geometry>
         </collision>
+        <xacro:inertial_cylinder mass="1.0" length="${j5_l}" radius="${j5_r}">
+            <origin xyz="${j5_xyz}" rpy="${j5_rpy}"/>
+        </xacro:inertial_cylinder>
     </link>
     <!-- j5 to flange Joint -->
@@ -268,6 +303,7 @@
         <parent link="j5_link"/>
         <child link="flange_link"/>
-    </joint>
-    <!-- The T link of the robot -->
+        <dynamics damping="${damping}" friction="${friction}" />
+    </joint>
+    <!-- The Flange link of the robot -->
     <link name="flange_link">
         <visual>
@@ -284,4 +320,7 @@
             </geometry>
         </collision>
+        <xacro:inertial_cylinder mass="1.0" length="${flange_l}" radius="${flange_r}">
+            <origin xyz="${flange_xyz}" rpy="${flange_rpy}"/>
+        </xacro:inertial_cylinder>
     </link>
 </robot>

Commit message: Add tcp support
- Changed from dbot.urdf.xacro to dbot_world.xacro

File: urdf/dbot.urdf.xacro (robot description, xacro)
@@ -324,3 +324,15 @@
         </xacro:inertial_cylinder>
     </link>
+    <!-- Load Tcp data -->
+    <xacro:property name="tcp_file" value="$(find dbot)/config/tcp.yaml"/>
+    <xacro:property name="tcp" value="${xacro.load_yaml(tcp_file)['tcp']}"/>
+    <!-- Flange to tcp -->
+    <joint name="tcp_joint" type="fixed">
+        <origin xyz="${tcp['x']} ${tcp['y']} ${tcp['z']}"
+                rpy="${tcp['roll']} ${tcp['pitch']} ${tcp['yaw']}"/>
+        <parent link="flange_link"/>
+        <child link="tcp_link"/>
+    </joint>
+    <!-- Tcp-->
+    <link name="tcp_link"/>
 </robot>

File: urdf/dbot_fake_hardware.urdf.xacro (robot description, xacro)
@@ -1,4 +1,4 @@
 <?xml version="1.0"?>
-<robot xmlns:xacro="http://www.ros.org/wiki/xacro" name="dbot">
+<robot xmlns:xacro="http://www.ros.org/wiki/xacro" name="dbot_fake">
     <!-- Import dbot urdf file -->
     <!-- <xacro:include filename="dbot.urdf.xacro"/> -->

File: urdf/dbot_gazebo.urdf.xacro (robot description, xacro)
@@ -1,4 +1,4 @@
 <?xml version="1.0"?>
-<robot xmlns:xacro="http://www.ros.org/wiki/xacro" name="dbot">
+<robot xmlns:xacro="http://www.ros.org/wiki/xacro" name="dbot_world">
     <!-- Import dbot urdf file -->
     <!-- <xacro:include filename="dbot.urdf.xacro"/> -->

File: urdf/dbot_world.xacro (robot description, xacro)
@@ -1,8 +1,8 @@
 <?xml version="1.0"?>
-<robot xmlns:xacro="http://www.ros.org/wiki/xacro">
+<robot xmlns:xacro="http://www.ros.org/wiki/xacro" name="dbot_world">
     <!-- World Frame-->
     <!-- Fixed base-->
     <link name="world"/>
-    <!-- - The upper limit uses xacro's mathematical features -->
+    <!-- World to robot base joint -->
     <joint name="world_base_joint" type="fixed">
         <origin xyz="0.0 0.0 0.0" rpy="0.0 0.0 0.0"/>
@@ -10,5 +10,5 @@
         <child link="base_link"/>
     </joint>
-    <!-- Commmon data for the robot. -->
+    <!-- Dbot robot urdf -->
     <xacro:include filename="dbot.urdf.xacro"/>
 </robot>
